File: LED-HeadBand.kicad_pcb (KiCad board)
At the start: 2 copper layers, 28 x 43.2 mm, 56 parts, among them J2 Screw_Terminal_01x03, Q1 PMOS, SW1 Mode_Switch, SW2 SW_DPDT_x2, U1 MAX9814, U2 RP2040, U3 W25Q16JVUXIQ_TR, U4 MIC5504-3.3YM5, U5 MCP73831-2-OT, U6 KH-TYPE-C-16P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

Commit message: Kristers man lika  mainīt lietas
Parts:
- R13: value 20k -> 50k
- R14: value 10k -> 100k
- turned R11 to 0 degrees
Connections:
- R12 pad 1: Net-(Q1-G) -> /MOSFET_Controll
Routing:
- net /MOSFET_Controll: track 10.7 -> 12.1 mm
Other:
- outline, holes or cut-outs redrawn
Changed lines of the file:
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@@
   )
   (footprint "Resistor_SMD:R_0402_1005Metric" (layer "F.Cu")
-    (at 139.192 30.607 180)
+    (at 139.192 30.607)
     (descr "Resistor SMD 0402 (1005 Metric), square (rectangular) end terminal, IPC_7351 nominal, (Body size source: IPC-SM-782 page 72, https://www.pcb-3d.com/wordpress/wp-content/uploads/ipc-sm-782a_amendment_1_and_2.pdf), generated with kicad-footprint-generator")
     (tags "resistor")
@@
     (property "ki_keywords" "R resistor")
     (attr smd)
-    (fp_text reference "R11" (at 0 -1.17 180) (layer "F.SilkS") hide
+    (fp_text reference "R11" (at 0 -1.17) (layer "F.SilkS") hide
         (effects (font (size 1 1) (thickness 0.15)))
     )
-    (fp_text value "300" (at 0 1.17 180) (layer "F.Fab")
+    (fp_text value "300" (at 0 1.17) (layer "F.Fab")
         (effects (font (size 1 1) (thickness 0.15)))
     )
-    (fp_text user "${REFERENCE}" (at 0 0 180) (layer "F.Fab")
+    (fp_text user "${REFERENCE}" (at 0 0) (layer "F.Fab")
         (effects (font (size 0.26 0.26) (thickness 0.04)))
     )
@@
     (fp_line (start 0.525 0.27) (end -0.525 0.27)
       (stroke (width 0.1) (type solid)) (layer "F.Fab"))
-    (pad "1" smd roundrect (at -0.51 0 180) (size 0.54 0.64) (layers "F.Cu" "F.Paste" "F.Mask") (roundrect_rratio 0.25)
+    (pad "1" smd roundrect (at -0.51 0) (size 0.54 0.64) (layers "F.Cu" "F.Paste" "F.Mask") (roundrect_rratio 0.25)
       (net 61 "/MOSFET_Controll") (pintype "passive"))
-    (pad "2" smd roundrect (at 0.51 0 180) (size 0.54 0.64) (layers "F.Cu" "F.Paste" "F.Mask") (roundrect_rratio 0.25)
+    (pad "2" smd roundrect (at 0.51 0) (size 0.54 0.64) (layers "F.Cu" "F.Paste" "F.Mask") (roundrect_rratio 0.25)
       (net 23 "Net-(Q1-G)") (pintype "passive"))
     (model "${KICAD6_3DMODEL_DIR}/Resistor_SMD.3dshapes/R_0402_1005Metric.wrl"
@@
         (effects (font (size 1 1) (thickness 0.15)))
     )
-    (fp_text value "20k" (at 0 1.17) (layer "F.Fab")
+    (fp_text value "50k" (at 0 1.17) (layer "F.Fab")
         (effects (font (size 1 1) (thickness 0.15)))
     )
@@
       (stroke (width 0.1) (type solid)) (layer "F.Fab"))
     (pad "1" smd roundrect (at -0.51 0 180) (size 0.54 0.64) (layers "F.Cu" "F.Paste" "F.Mask") (roundrect_rratio 0.25)
-      (net 23 "Net-(Q1-G)") (pintype "passive"))
+      (net 61 "/MOSFET_Controll") (pintype "passive"))
     (pad "2" smd roundrect (at 0.51 0 180) (size 0.54 0.64) (layers "F.Cu" "F.Paste" "F.Mask") (roundrect_rratio 0.25)
       (net 16 "+BATT") (pintype "passive"))
@@
         (effects (font (size 1 1) (thickness 0.15)))
     )
-    (fp_text value "10k" (at 0 1.17) (layer "F.Fab")
+    (fp_text value "100k" (at 0 1.17) (layer "F.Fab")
         (effects (font (size 1 1) (thickness 0.15)))
     )
@@
   (gr_line (start 152 58.539) (end 124 58.539)
     (stroke (width 0.1) (type default)) (layer "Edge.Cuts"))
-  (gr_line (start 145.288 15.367) (end 136.017 15.367)
+  (gr_line (start 145.288 15.367) (end 134.239 15.367)
     (stroke (width 0.1) (type default)) (layer "Edge.Cuts"))
   (gr_arc (start 149.479 25.4) (mid 146.515515 24.172485) (end 145.288 21.209)
     (stroke (width 0.1) (type default)) (layer "Edge.Cuts"))
-  (gr_arc (start 136.017 21.209) (mid 134.789485 24.172485) (end 131.826 25.4)
+  (gr_arc (start 134.239 21.209) (mid 133.011485 24.172485) (end 130.048 25.4)
     (stroke (width 0.1) (type default)) (layer "Edge.Cuts"))
   (gr_line (start 145.288 15.367) (end 145.288 21.209)
     (stroke (width 0.1) (type default)) (layer "Edge.Cuts"))
-  (gr_line (start 136.017 21.209) (end 136.017 15.367)
+  (gr_line (start 134.239 21.209) (end 134.239 15.367)
+    (stroke (width 0.1) (type default)) (layer "Edge.Cuts"))
+  (gr_line (start 130.048 25.4) (end 124 25.4)
     (stroke (width 0.1) (type default)) (layer "Edge.Cuts"))
   (gr_line (start 124 58.539) (end 124 25.4)
@@
   (gr_line (start 149.479 25.4) (end 152 25.4)
     (stroke (width 0.1) (type default)) (layer "Edge.Cuts"))
-  (gr_line (start 131.826 25.4) (end 124 25.4)
-    (stroke (width 0.1) (type default)) (layer "Edge.Cuts"))
   (gr_text "-" (at 124.0536 29.464) (layer "B.SilkS")
     (effects (font (size 1 1) (thickness 0.15)) (justify left bottom))
@@
   (via (at 142.113 42.799) (size 0.6) (drill 0.4) (layers "F.Cu" "B.Cu") (net 1))
   (via (at 140.081 42.799) (size 0.6) (drill 0.4) (layers "F.Cu" "B.Cu") (net 1))
-  (via (at 145.542 48.26) (size 0.6) (drill 0.4) (layers "F.Cu" "B.Cu") (free) (net 1))
+  (via (at 145.542 47.879) (size 0.6) (drill 0.4) (layers "F.Cu" "B.Cu") (free) (net 1))
   (via (at 146.812 40.64) (size 0.6) (drill 0.4) (layers "F.Cu" "B.Cu") (free) (net 1))
   (via (at 136.525 31.369) (size 0.6) (drill 0.4) (layers "F.Cu" "B.Cu") (free) (net 1))
@@
   (segment (start 145.348 41.977) (end 144.4965 41.977) (width 0.2) (layer "F.Cu") (net 2))
   (segment (start 146.6685 39.497) (end 146.2645 39.497) (width 0.2) (layer "F.Cu") (net 2))
-  (segment (start 146.6685 39.1325) (end 146.179 39.1325) (width 0.15) (layer "F.Cu") (net 3))
   (segment (start 145.136 41.375) (end 144.934 41.577) (width 0.15) (layer "F.Cu") (net 3))
-  (segment (start 146.6685 38.997) (end 146.6685 39.1325) (width 0.15) (layer "F.Cu") (net 3))
-  (segment (start 145.136 40.1755) (end 145.136 41.375) (width 0.15) (layer "F.Cu") (net 3))
+  (segment (start 146.337408 38.997) (end 145.136 40.198408) (width 0.15) (layer "F.Cu") (net 3))
+  (segment (start 146.6685 38.997) (end 146.337408 38.997) (width 0.15) (layer "F.Cu") (net 3))
+  (segment (start 145.136 40.198408) (end 145.136 41.375) (width 0.15) (layer "F.Cu") (net 3))
   (segment (start 144.934 41.577) (end 144.4965 41.577) (width 0.15) (layer "F.Cu") (net 3))
-  (segment (start 146.179 39.1325) (end 145.136 40.1755) (width 0.15) (layer "F.Cu") (net 3))
   (segment (start 145.415 37.34) (end 146.431 37.34) (width 0.15) (layer "F.Cu") (net 4))
   (segment (start 146.6685 38.497) (end 146.6685 37.5775) (width 0.15) (layer "F.Cu") (net 4))
@@
   (segment (start 140.225 36.0645) (end 140.225 27.49) (width 0.2) (layer "B.Cu") (net 22))
   (segment (start 133.6396 26.7826) (end 134.7614 26.7826) (width 0.2) (layer "F.Cu") (net 23))
+  (segment (start 139.573 31.623) (end 139.573 30.736) (width 0.2) (layer "F.Cu") (net 23))
   (segment (start 134.7614 26.7826) (end 135.255 26.289) (width 0.2) (layer "F.Cu") (net 23))
-  (segment (start 138.176 31.093) (end 137.69 30.607) (width 0.2) (layer "F.Cu") (net 23))
-  (segment (start 138.176 31.75) (end 138.176 31.093) (width 0.2) (layer "F.Cu") (net 23))
-  (segment (start 137.69 30.607) (end 138.682 30.607) (width 0.2) (layer "F.Cu") (net 23))
+  (segment (start 139.573 30.736) (end 139.702 30.607) (width 0.2) (layer "F.Cu") (net 23))
   (via (at 135.255 26.289) (size 0.6) (drill 0.4) (layers "F.Cu" "B.Cu") (net 23))
-  (via (at 138.176 31.75) (size 0.6) (drill 0.4) (layers "F.Cu" "B.Cu") (net 23))
-  (segment (start 135.255 26.289) (end 135.255 28.829) (width 0.2) (layer "B.Cu") (net 23))
-  (segment (start 135.255 28.829) (end 138.176 31.75) (width 0.2) (layer "B.Cu") (net 23))
+  (via (at 139.573 31.623) (size 0.6) (drill 0.4) (layers "F.Cu" "B.Cu") (net 23))
+  (segment (start 139.573 31.623) (end 138.049 31.623) (width 0.2) (layer "B.Cu") (net 23))
+  (segment (start 138.049 31.623) (end 135.255 28.829) (width 0.2) (layer "B.Cu") (net 23))
+  (segment (start 135.255 28.829) (end 135.255 26.289) (width 0.2) (layer "B.Cu") (net 23))
   (segment (start 145.832 52.036) (end 145.832 50.598) (width 0.2) (layer "F.Cu") (net 24))
   (segment (start 143.258 54.61) (end 143.637 54.231) (width 0.2) (layer "F.Cu") (net 24))
@@
   (segment (start 139.558 51.5335) (end 138.5285 51.5335) (width 0.15) (layer "F.Cu") (net 57))
   (segment (start 138.5285 51.5335) (end 137.767 50.772) (width 0.15) (layer "F.Cu") (net 57))
+  (segment (start 139.046 33.251) (end 139.046 30.971) (width 0.2) (layer "F.Cu") (net 61))
   (segment (start 142.059 39.697) (end 142.059 40.3395) (width 0.2) (layer "F.Cu") (net 61))
   (segment (start 139.702 37.34) (end 142.059 39.697) (width 0.2) (layer "F.Cu") (net 61))
-  (segment (start 139.702 30.607) (end 139.702 37.34) (width 0.2) (layer "F.Cu") (net 61))
+  (segment (start 139.702 37.34) (end 139.702 33.907) (width 0.2) (layer "F.Cu") (net 61))
+  (segment (start 137.69 30.607) (end 138.682 30.607) (width 0.25) (layer "F.Cu") (net 61))
+  (segment (start 139.046 30.971) (end 138.682 30.607) (width 0.2) (layer "F.Cu") (net 61))
+  (segment (start 139.702 33.907) (end 139.046 33.251) (width 0.2) (layer "F.Cu") (net 61))
   (segment (start 132.6896 29.0576) (end 141.1804 29.0576) (width 0.5) (layer "F.Cu") (net 62))
   (segment (start 141.1804 29.0576) (end 142.748 27.49) (width 0.5) (layer "F.Cu") (net 62))
