File: LED-HeadBand.kicad_sch (KiCad schematic)
At the start: 56 parts, among them J2 Screw_Terminal_01x03, Q1 PMOS, SW1 Mode_Switch, SW2 SW_DPDT_x2, U1 MAX9814, U2 RP2040, U3 W25Q16JVUXIQ_TR, U4 MIC5504-3.3YM5, U5 MCP73831-2-OT, U6 KH-TYPE-C-16P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

Commit message: Kristers man lika  mainīt lietas
Parts:
- R13: value 20k -> 50k
- R14: value 10k -> 100k
Connections:
- net MOSFET_Controll: now also R15.1
- net at Q1.1 (G), R14.2: no longer R15.1
Other:
- moved on the sheet: R15
Changed lines of the file:
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@@
   (junction (at 55.118 38.354) (diameter 0) (color 0 0 0 0)
   )
-  (junction (at 142.875 171.45) (diameter 0) (color 0 0 0 0)
-  )
   (junction (at 243.205 41.275) (diameter 0) (color 0 0 0 0)
   )
@@
   (junction (at 250.825 60.325) (diameter 0) (color 0 0 0 0)
   )
+  (junction (at 135.255 171.45) (diameter 0) (color 0 0 0 0)
+  )
   (junction (at 40.64 186.69) (diameter 0) (color 0 0 0 0)
   )
@@
     (stroke (width 0) (type default))
   )
-  (wire (pts (xy 142.875 164.465) (xy 142.875 171.45))
+  (wire (pts (xy 135.255 164.465) (xy 135.255 171.45))
     (stroke (width 0) (type default))
   )
@@
     (stroke (width 0) (type default))
   )
-  (wire (pts (xy 141.605 171.45) (xy 142.875 171.45))
-    (stroke (width 0) (type default))
-  )
   (wire (pts (xy 243.205 59.055) (xy 243.205 63.5))
     (stroke (width 0) (type default))
@@
     (stroke (width 0) (type default))
   )
-  (wire (pts (xy 130.81 171.45) (xy 136.525 171.45))
+  (wire (pts (xy 130.81 171.45) (xy 135.255 171.45))
     (stroke (width 0) (type default))
   )
@@
     (stroke (width 0) (type default))
   )
-  (wire (pts (xy 142.875 158.115) (xy 142.875 159.385))
+  (wire (pts (xy 135.255 158.115) (xy 135.255 159.385))
     (stroke (width 0) (type default))
   )
@@
     (stroke (width 0) (type default))
   )
+  (wire (pts (xy 135.255 171.45) (xy 136.525 171.45))
+    (stroke (width 0) (type default))
+  )
   (wire (pts (xy 149.86 40.64) (xy 151.765 40.64))
     (stroke (width 0) (type default))
   )
-  (wire (pts (xy 142.875 171.45) (xy 144.78 171.45))
+  (wire (pts (xy 141.605 171.45) (xy 144.78 171.45))
     (stroke (width 0) (type default))
   )
@@
       (effects (font (size 1.27 1.27)) (justify left))
     )
-    (property "Value" "10k" (at 177.8 152.146 0)
+    (property "Value" "100k" (at 177.8 152.146 0)
       (effects (font (size 1.27 1.27)) (justify left))
     )
@@
       (effects (font (size 1.27 1.27)) (justify left))
     )
-    (property "Value" "20k" (at 177.8 144.018 0)
+    (property "Value" "50k" (at 177.8 144.018 0)
       (effects (font (size 1.27 1.27)) (justify left))
     )
@@
     )
   )
-  (symbol (lib_id "Device:R_Small") (at 142.875 161.925 180) (unit 1)
+  (symbol (lib_id "Device:R_Small") (at 135.255 161.925 180) (unit 1)
     (in_bom yes) (on_board yes) (dnp no)
-    (property "Reference" "R15" (at 137.795 161.29 0)
+    (property "Reference" "R15" (at 130.175 161.29 0)
       (effects (font (size 1.27 1.27)) (justify right))
     )
-    (property "Value" "10k" (at 137.16 163.195 0)
+    (property "Value" "10k" (at 129.54 163.195 0)
       (effects (font (size 1.27 1.27)) (justify right))
     )
-    (property "Footprint" "Resistor_SMD:R_0402_1005Metric" (at 142.875 161.925 0)
+    (property "Footprint" "Resistor_SMD:R_0402_1005Metric" (at 135.255 161.925 0)
       (effects (font (size 1.27 1.27)) hide)
     )
-    (property "Datasheet" "~" (at 142.875 161.925 0)
+    (property "Datasheet" "~" (at 135.255 161.925 0)
       (effects (font (size 1.27 1.27)) hide)
     )
@@
     )
   )
-  (symbol (lib_id "power:+BATT") (at 142.875 158.115 0) (unit 1)
+  (symbol (lib_id "power:+BATT") (at 135.255 158.115 0) (unit 1)
     (in_bom yes) (on_board yes) (dnp no)
-    (property "Reference" "#PWR028" (at 142.875 161.925 0)
+    (property "Reference" "#PWR028" (at 135.255 161.925 0)
       (effects (font (size 1.27 1.27)) hide)
     )
-    (property "Value" "+BATT" (at 139.065 154.94 0)
+    (property "Value" "+BATT" (at 131.445 154.94 0)
       (effects (font (size 1.27 1.27)))
     )
-    (property "Footprint" "" (at 142.875 158.115 0)
+    (property "Footprint" "" (at 135.255 158.115 0)
       (effects (font (size 1.27 1.27)) hide)
     )
-    (property "Datasheet" "" (at 142.875 158.115 0)
+    (property "Datasheet" "" (at 135.255 158.115 0)
       (effects (font (size 1.27 1.27)) hide)
     )
